File: Circuit_design/Circuit.sch (EAGLE design)
At the start: 42 parts, among them IC1 LM358D, IC2 LM358D, IC3 LM358D, IC4 LM358D, IC5 LM358D, IC6 LM358D

Commit message: Add updates
Parts:
- R11, R12, R15, R16, R19, R20, R23, R24, R3, R4, R7, R8: value 100 -> 4700
Changed lines of the file:
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@@
 <part name="P+1" library="supply1" library_urn="urn:adsk.eagle:library:371" deviceset="+5V" device=""/>
 <part name="IC1" library="linear" library_urn="urn:adsk.eagle:library:262" deviceset="LM358" device="D"/>
-<part name="R3" library="rcl" library_urn="urn:adsk.eagle:library:334" deviceset="R-EU_" device="0204/2V" value="100"/>
-<part name="R4" library="rcl" library_urn="urn:adsk.eagle:library:334" deviceset="R-EU_" device="0204/2V" value="100"/>
+<part name="R3" library="rcl" library_urn="urn:adsk.eagle:library:334" deviceset="R-EU_" device="0204/2V" value="4700"/>
+<part name="R4" library="rcl" library_urn="urn:adsk.eagle:library:334" deviceset="R-EU_" device="0204/2V" value="4700"/>
 <part name="P+2" library="supply1" library_urn="urn:adsk.eagle:library:371" deviceset="+5V" device=""/>
 <part name="GND2" library="supply1" library_urn="urn:adsk.eagle:library:371" deviceset="GND" device=""/>
@@
 <part name="P+3" library="supply1" library_urn="urn:adsk.eagle:library:371" deviceset="+5V" device=""/>
 <part name="IC2" library="linear" library_urn="urn:adsk.eagle:library:262" deviceset="LM358" device="D"/>
-<part name="R7" library="rcl" library_urn="urn:adsk.eagle:library:334" deviceset="R-EU_" device="0204/2V" value="100"/>
-<part name="R8" library="rcl" library_urn="urn:adsk.eagle:library:334" deviceset="R-EU_" device="0204/2V" value="100"/>
+<part name="R7" library="rcl" library_urn="urn:adsk.eagle:library:334" deviceset="R-EU_" device="0204/2V" value="4700"/>
+<part name="R8" library="rcl" library_urn="urn:adsk.eagle:library:334" deviceset="R-EU_" device="0204/2V" value="4700"/>
 <part name="P+4" library="supply1" library_urn="urn:adsk.eagle:library:371" deviceset="+5V" device=""/>
 <part name="GND4" library="supply1" library_urn="urn:adsk.eagle:library:371" deviceset="GND" device=""/>
@@
 <part name="P+5" library="supply1" library_urn="urn:adsk.eagle:library:371" deviceset="+5V" device=""/>
 <part name="IC3" library="linear" library_urn="urn:adsk.eagle:library:262" deviceset="LM358" device="D"/>
-<part name="R11" library="rcl" library_urn="urn:adsk.eagle:library:334" deviceset="R-EU_" device="0204/2V" value="100"/>
-<part name="R12" library="rcl" library_urn="urn:adsk.eagle:library:334" deviceset="R-EU_" device="0204/2V" value="100"/>
+<part name="R11" library="rcl" library_urn="urn:adsk.eagle:library:334" deviceset="R-EU_" device="0204/2V" value="4700"/>
+<part name="R12" library="rcl" library_urn="urn:adsk.eagle:library:334" deviceset="R-EU_" device="0204/2V" value="4700"/>
 <part name="P+6" library="supply1" library_urn="urn:adsk.eagle:library:371" deviceset="+5V" device=""/>
 <part name="GND6" library="supply1" library_urn="urn:adsk.eagle:library:371" deviceset="GND" device=""/>
@@
 <part name="P+7" library="supply1" library_urn="urn:adsk.eagle:library:371" deviceset="+5V" device=""/>
 <part name="IC4" library="linear" library_urn="urn:adsk.eagle:library:262" deviceset="LM358" device="D"/>
-<part name="R15" library="rcl" library_urn="urn:adsk.eagle:library:334" deviceset="R-EU_" device="0204/2V" value="100"/>
-<part name="R16" library="rcl" library_urn="urn:adsk.eagle:library:334" deviceset="R-EU_" device="0204/2V" value="100"/>
+<part name="R15" library="rcl" library_urn="urn:adsk.eagle:library:334" deviceset="R-EU_" device="0204/2V" value="4700"/>
+<part name="R16" library="rcl" library_urn="urn:adsk.eagle:library:334" deviceset="R-EU_" device="0204/2V" value="4700"/>
 <part name="P+8" library="supply1" library_urn="urn:adsk.eagle:library:371" deviceset="+5V" device=""/>
 <part name="GND8" library="supply1" library_urn="urn:adsk.eagle:library:371" deviceset="GND" device=""/>
@@
 <part name="P+9" library="supply1" library_urn="urn:adsk.eagle:library:371" deviceset="+5V" device=""/>
 <part name="IC5" library="linear" library_urn="urn:adsk.eagle:library:262" deviceset="LM358" device="D"/>
-<part name="R19" library="rcl" library_urn="urn:adsk.eagle:library:334" deviceset="R-EU_" device="0204/2V" value="100"/>
-<part name="R20" library="rcl" library_urn="urn:adsk.eagle:library:334" deviceset="R-EU_" device="0204/2V" value="100"/>
+<part name="R19" library="rcl" library_urn="urn:adsk.eagle:library:334" deviceset="R-EU_" device="0204/2V" value="4700"/>
+<part name="R20" library="rcl" library_urn="urn:adsk.eagle:library:334" deviceset="R-EU_" device="0204/2V" value="4700"/>
 <part name="P+10" library="supply1" library_urn="urn:adsk.eagle:library:371" deviceset="+5V" device=""/>
 <part name="GND10" library="supply1" library_urn="urn:adsk.eagle:library:371" deviceset="GND" device=""/>
@@
 <part name="P+11" library="supply1" library_urn="urn:adsk.eagle:library:371" deviceset="+5V" device=""/>
 <part name="IC6" library="linear" library_urn="urn:adsk.eagle:library:262" deviceset="LM358" device="D"/>
-<part name="R23" library="rcl" library_urn="urn:adsk.eagle:library:334" deviceset="R-EU_" device="0204/2V" value="100"/>
-<part name="R24" library="rcl" library_urn="urn:adsk.eagle:library:334" deviceset="R-EU_" device="0204/2V" value="100"/>
+<part name="R23" library="rcl" library_urn="urn:adsk.eagle:library:334" deviceset="R-EU_" device="0204/2V" value="4700"/>
+<part name="R24" library="rcl" library_urn="urn:adsk.eagle:library:334" deviceset="R-EU_" device="0204/2V" value="4700"/>
 <part name="P+12" library="supply1" library_urn="urn:adsk.eagle:library:371" deviceset="+5V" device=""/>
 <part name="GND12" library="supply1" library_urn="urn:adsk.eagle:library:371" deviceset="GND" device=""/>

Commit message: Change circuit info
Parts:
- added D13, D15, D17, D19, D21, D23, D25, D27, D29, D31, D33, D35, D37, D39, D41, D43, D45, D47: BP104, opto-trans-siemens:BP104
- added D14, D16, D18, D20, D22, D24, D26, D28, D30, D32, D34, D36, D38, D40, D42, D44, D46, D48: HLMP6, display-hp:HLMP6
- added IC10, IC11, IC12, IC13, IC14, IC15, IC16, IC17, IC18, IC19, IC20, IC21, IC22, IC23, IC24, IC7, IC8, IC9: LM358D, linear:LM358D
- added J_ULTRASONIC_1, J_ULTRASONIC_2: HC-SR04, Ultrasonic-sensor:HC-SR04
- added R25, R29, R33, R37, R41, R45, R49, R53, R57, R61, R65, R69, R73, R77, R81, R85, R89, R93: 10000, rcl:R-EU_0204/2V
- added R26, R30, R34, R38, R42, R46, R50, R54, R58, R62, R66, R70, R74, R78, R82, R86, R90, R94: 100, rcl:R-EU_0204/2V
- added R27, R28, R31, R32, R35, R36, R39, R40, R43, R44, R47, R48, R51, R52, R55, R56, R59, R60, R63, R64, R67, R68, R71, R72, R75, R76, R79, R80, R83, R84, R87, R88, R91, R92, R95, R96: 4700, rcl:R-EU_0204/2V
Connections:
- new net N$19: D13.A, IC7A.-IN, R25.1
- new net N$20: IC7A.+IN, R27.1, R28.1
- new net N$21: D14.K, R26.1
- new net N$22: D15.A, IC8A.-IN, R29.1
- new net N$23: IC8A.+IN, R31.1, R32.1
- new net N$24: D16.K, R30.1
- new net N$25: D17.A, IC9A.-IN, R33.1
- new net N$26: IC9A.+IN, R35.1, R36.1
- new net N$27: D18.K, R34.1
- new net N$28: D19.A, IC10A.-IN, R37.1
- new net N$29: IC10A.+IN, R39.1, R40.1
- new net N$30: D20.K, R38.1
- new net N$31: D21.A, IC11A.-IN, R41.1
- new net N$32: IC11A.+IN, R43.1, R44.1
- new net N$33: D22.K, R42.1
- new net N$34: D23.A, IC12A.-IN, R45.1
- new net N$35: IC12A.+IN, R47.1, R48.1
- new net N$36: D24.K, R46.1
- new net N$37: D25.A, IC13A.-IN, R49.1
- new net N$38: IC13A.+IN, R51.1, R52.1
- new net N$39: D26.K, R50.1
- new net N$40: D27.A, IC14A.-IN, R53.1
- new net N$41: IC14A.+IN, R55.1, R56.1
- new net N$42: D28.K, R54.1
- new net N$43: D29.A, IC15A.-IN, R57.1
- new net N$44: IC15A.+IN, R59.1, R60.1
- new net N$45: D30.K, R58.1
- new net N$46: D31.A, IC16A.-IN, R61.1
- new net N$47: IC16A.+IN, R63.1, R64.1
- new net N$48: D32.K, R62.1
- new net N$49: D33.A, IC17A.-IN, R65.1
- new net N$50: IC17A.+IN, R67.1, R68.1
- new net N$51: D34.K, R66.1
- new net N$52: D35.A, IC18A.-IN, R69.1
- new net N$53: IC18A.+IN, R71.1, R72.1
- new net N$54: D36.K, R70.1
- new net N$55: D37.A, IC19A.-IN, R73.1
- new net N$56: IC19A.+IN, R75.1, R76.1
- new net N$57: D38.K, R74.1
- new net N$58: D39.A, IC20A.-IN, R77.1
- new net N$59: IC20A.+IN, R79.1, R80.1
- new net N$60: D40.K, R78.1
- new net N$61: D41.A, IC21A.-IN, R81.1
- new net N$62: IC21A.+IN, R83.1, R84.1
- new net N$63: D42.K, R82.1
- new net N$64: D43.A, IC22A.-IN, R85.1
- new net N$65: IC22A.+IN, R87.1, R88.1
- new net N$66: D44.K, R86.1
- new net N$67: D45.A, IC23A.-IN, R89.1
- new net N$68: IC23A.+IN, R91.1, R92.1
- new net N$69: D46.K, R90.1
- new net N$70: D47.A, IC24A.-IN, R93.1
- new net N$71: IC24A.+IN, R95.1, R96.1
- new net N$72: D48.K, R94.1
- net +5V: now also D13.C, D14.A, D15.C, D16.A, D17.C, D18.A, D19.C, D20.A, D21.C, D22.A, D23.C, D24.A, D25.C, D26.A, D27.C, D28.A, D29.C, D30.A, D31.C, D32.A, D33.C, D34.A, D35.C, D36.A, D37.C, D38.A, D39.C, D40.A, D41.C, D42.A, D43.C, D44.A, D45.C, D46.A, D47.C, D48.A, J_ULTRASONIC_1.5V, J_ULTRASONIC_2.5V, R28.2, R32.2, R36.2, R40.2, R44.2, R48.2, R52.2, R56.2, R60.2, R64.2, R68.2, R72.2, R76.2, R80.2, R84.2, R88.2, R92.2, R96.2
- net GND: now also J_ULTRASONIC_1.GND, J_ULTRASONIC_2.GND, R25.2, R26.2, R27.2, R29.2, R30.2, R31.2, R33.2, R34.2, R35.2, R37.2, R38.2, R39.2, R41.2, R42.2, R43.2, R45.2, R46.2, R47.2, R49.2, R50.2, R51.2, R53.2, R54.2, R55.2, R57.2, R58.2, R59.2, R61.2, R62.2, R63.2, R65.2, R66.2, R67.2, R69.2, R70.2, R71.2, R73.2, R74.2, R75.2, R77.2, R78.2, R79.2, R81.2, R82.2, R83.2, R85.2, R86.2, R87.2, R89.2, R90.2, R91.2, R93.2, R94.2, R95.2
Other:
- moved on the sheet: D1, D10, D11, D12, D2, D3, D4, D5, D6, D7, D8, D9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

Commit message: Add shift register and modify circuit
Parts:
- removed IC1, IC10, IC11, IC12, IC2, IC3, IC4, IC5, IC6, IC7, IC8, IC9: LM358D, linear:LM358D
- removed R11, R12, R15, R16, R19, R20, R23, R24, R27, R28, R3, R31, R32, R35, R36, R39, R4, R40, R43, R44, R47, R48, R7, R8: 4700, rcl:R-EU_0204/2V
- added IC25: ATMEGA328-20P, atmega328:ATMEGA328-20P
- added IC26, IC27: 4014D, 40xx:4014D
- added Q1: (no value), special:XTAL
- added U$1: RELAYPTH, relay:RELAYPTH
Connections:
- removed net N$11: IC4A.+IN, R15.1, R16.1
- removed net N$14: IC5A.+IN, R19.1, R20.1
- removed net N$17: IC6A.+IN, R23.1, R24.1
- removed net N$19: D13.A, IC7A.-IN, R25.1
- removed net N$20: IC7A.+IN, R27.1, R28.1
- removed net N$22: D15.A, IC8A.-IN, R29.1
- removed net N$23: IC8A.+IN, R31.1, R32.1
- removed net N$26: IC9A.+IN, R35.1, R36.1
- removed net N$28: D19.A, IC10A.-IN, R37.1
- removed net N$3: IC1A.+IN, R3.1, R4.1
- removed net N$35: IC12A.+IN, R47.1, R48.1
- removed net N$37: D25.A, IC13A.-IN, R49.1
- removed net N$40: D27.A, IC14A.-IN, R53.1
- removed net N$46: D31.A, IC16A.-IN, R61.1
- removed net N$5: IC2A.+IN, R7.1, R8.1
- removed net N$55: D37.A, IC19A.-IN, R73.1
- removed net N$58: D39.A, IC20A.-IN, R77.1
- removed net N$61: D41.A, IC21A.-IN, R81.1
- removed net N$64: D43.A, IC22A.-IN, R85.1
- removed net N$67: D45.A, IC23A.-IN, R89.1
- removed net N$70: D47.A, IC24A.-IN, R93.1
- removed net N$8: IC3A.+IN, R11.1, R12.1
- new net CLK: IC25.(PCI23/AIN1)PD7
- new net ECHO: IC25.(PCI17/TXD)PD1, IC25.(PCI19/INT1/OC2B)PD3
- new net N$73: IC26A.P1, IC27A.P1
- new net N$74: IC26A.P2, IC27A.P2
- new net N$75: IC26A.P3, IC27A.P3
- new net N$76: IC26A.P/!S
- new net N$77: IC26A.P4, IC27A.P4
- new net N$78: IC26A.P5, IC27A.P5
- new net N$79: IC26A.P6, IC27A.P6
- new net N$80: IC26A.P7, IC27A.P7
- new net N$81: IC27A.P/!S
- new net N$82: IC26A.SI, IC27A.Q7
- new net P/S: IC25.(PCI0/ICP/CLKO)PB0
- new net P1: IC18A.OUT
- new net P10: IC21A.OUT
- new net P11: IC20A.OUT
- new net P12: IC19A.OUT
- new net P2: IC17A.OUT
- new net P3: IC16A.OUT
- new net P4: IC15A.OUT
- new net P5: IC14A.OUT
- new net P6: IC13A.OUT
- new net P7: IC24A.OUT
- new net P8: IC23A.OUT
- new net P9: IC22A.OUT
- new net PB0: IC26A.CLK, IC27A.CLK
- new net PB1: IC26A.Q8, IC27A.Q8
- new net PB5: U$1.COIL1
- new net PD0: J_ULTRASONIC_1.TRIG
- new net PD1: J_ULTRASONIC_1.ECHO
- new net PD2: J_ULTRASONIC_2.TRIG
- new net PD3: J_ULTRASONIC_2.ECHO
- new net Q8: IC25.(PCI1/OC1A/OC1S)PB1
- new net RELAY: IC25.(PCI5/SCK)PB5
- new net TRIGG: IC25.(PCI16/RXD)PD0, IC25.(PCI18/INT0)PD2
- net +5V: now also IC25.GND, U$1.SWCOMMON; no longer D1.C, D10.A, D11.C, D12.A, D13.C, D14.A, D15.C, D16.A, D17.C, D18.A, D19.C, D2.C, D20.A, D21.C, D22.A, D23.C, D24.A, D25.C, D26.A, D27.C, D28.A, D29.C, D3.A, D30.A, D31.C, D32.A, D33.C, D34.A, D35.C, D36.A, D37.C, D38.A, D39.C, D4.C, D40.A, D41.C, D42.A, D43.C, D44.A, D45.C, D46.A, D47.C, D48.A, D5.A, D6.C, D7.A, D8.A, D9.C, R12.2, R16.2, R20.2, R24.2, R28.2, R32.2, R36.2, R4.2, R40.2, R44.2, R48.2, R8.2
- net GND: now also IC25.PB6(XTAL1/TOSC1/PCI6), IC25.PB7(XTAL2/TOSC2/PCI7), IC25.VCC, Q1.1, Q1.2, U$1.COIL0; no longer R11.2, R15.2, R19.2, R23.2, R27.2, R3.2, R31.2, R35.2, R39.2, R43.2, R47.2, R7.2
- net N$1: now also D45.A, IC23A.-IN, R89.1; no longer IC2A.-IN
- net N$10: now also D41.A, IC21A.-IN, R81.1; no longer IC4A.-IN
- net N$13: now also D39.A, IC20A.-IN, R77.1; no longer IC5A.-IN
- net N$16: now also D37.A, IC19A.-IN, R73.1; no longer IC6A.-IN
- net N$2: now also D47.A, IC24A.-IN, R93.1; no longer IC1A.-IN
- net N$25: now also D31.A, IC16A.-IN, R61.1; no longer IC9A.-IN
- net N$29: now also D25.C, D26.A, D27.C, D28.A, D29.C, D30.A, D31.C, D32.A, D33.C, D34.A, D35.C, D36.A, D37.C, D38.A, D39.C, D40.A, D41.C, D42.A, D43.C, D44.A, D45.C, D46.A, D47.C, D48.A, U$1.SWOPEN; no longer IC10A.+IN, R39.1, R40.1
- net N$31: now also D27.A, IC14A.-IN, R53.1; no longer IC11A.-IN
- net N$32: now also D1.C, D10.A, D11.C, D12.A, D13.C, D14.A, D15.C, D16.A, D17.C, D18.A, D19.C, D2.C, D20.A, D21.C, D22.A, D23.C, D24.A, D3.A, D4.C, D5.A, D6.C, D7.A, D8.A, D9.C, U$1.SWCLOSE; no longer IC11A.+IN, R43.1, R44.1
- net N$34: now also D25.A, IC13A.-IN, R49.1; no longer IC12A.-IN
- net N$43: now also D19.A, R37.1
- net N$49: now also D15.A, R29.1
- net N$52: now also D13.A, R25.1
- net N$7: now also D43.A, IC22A.-IN, R85.1; no longer IC3A.-IN

Commit message: Clean up changes with the circuit
Connections:
- removed net N$73: IC26A.P1, IC27A.P1
- removed net N$74: IC26A.P2, IC27A.P2
- removed net N$75: IC26A.P3, IC27A.P3
- removed net N$77: IC26A.P4, IC27A.P4
- removed net N$78: IC26A.P5, IC27A.P5
- removed net N$79: IC26A.P6, IC27A.P6
- removed net N$80: IC26A.P7, IC27A.P7
- new net OUTPUT0: IC26A.P1
- new net OUTPUT1: IC26A.P2
- new net OUTPUT10: IC27A.P3
- new net OUTPUT11: IC27A.P4
- new net OUTPUT2: IC26A.P3
- new net OUTPUT3: IC26A.P4
- new net OUTPUT4: IC26A.P5
- new net OUTPUT5: IC26A.P6
- new net OUTPUT6: IC26A.P7
- new net OUTPUT7: IC26A.P8
- new net OUTPUT8: IC27A.P1
- new net OUTPUT9: IC27A.P2
Other:
- moved on the sheet: IC25, Q1
